Commit message: additional tuning needed

File: drake/examples/kuka_iiwa_arm/models/objects/block_for_pick_and_place.urdf (robot description, URDF)
Before this commit: robot simple_cuboid, 1 links, 0 joints
Links:
- link base_link: geometry collision box size=0.029 0.029 0.199; collision sphere radius=1e-7

Commit message: works

File: drake/examples/kuka_iiwa_arm/models/objects/block_for_pick_and_place.urdf (robot description, URDF)
Before this commit: robot simple_cuboid, 1 links, 0 joints
Links:
- link base_link: geometry collision box size=0.059 0.029 0.199; collision sphere radius=1e-7

File: drake/manipulation/models/gelsight_description/urdf/simple_gelsight.urdf (robot description, URDF)
Before this commit: robot gelsight_sensor, 2 links, 1 joints
Links:
- link gelsight_base_link: geometry collision cylinder length=0.02 radius=0.02; visual cylinder length=0.02 radius=0.02
- link gelsight_camera_head: geometry collision sphere radius=0.015; visual sphere radius=0.017
Joints:
- joint gelsight_camera_joint: origin xyz=0 0.0 0 rpy=0 0 0 -> xyz=0.0 0.00 0 rpy=0 0 0
