Commit message: mesh model to box

File: drake/manipulation/models/gelsight_description/urdf/simple_gelsight.urdf (robot description, URDF)
Before this commit: robot gelsight_sensor, 2 links, 1 joints
Links:
- link gelsight_camera_head: geometry collision sphere radius=0.017; visual sphere radius=0.017
